File: BufferedMult_bottom.kicad_pcb (KiCad board)
At the start: 2 copper layers, 24.8 x 68.6 mm, 23 parts, among them J1 Conn_01x05_Male, J2 Conn_01x05_Male, J3 Conn_02x05_Odd_Even, U1 TL074, U2 TL074

Commit message: Add files via upload
Parts:
- D1, D2: value 1N4148 -> 1N5817; footprint Diode_THT:D_DO-35_SOD27_P7.62mm_Horizontal -> Diode_THT:D_DO-41_SOD81_P10.16mm_Horizontal
- moved C1 4.30 mm to (37.8, 132.3), turned to 270 degrees
- moved FB2 3.18 mm to (49.3, 138.5)
- moved FB1 3.16 mm to (49.3, 134.2)
- moved C2 3.08 mm to (37.8, 138.1), turned to 270 degrees
- moved D1 2.92 mm to (41.9, 131.1)
- moved D2 0.50 mm to (52.1, 141.6)
Routing:
- net +12V: track 76.1 -> 86.4 mm, vias 4 -> 2
- net -12V: track 71.5 -> 77.9 mm
Other:
- board text added: "-12V"
- board text removed: "Stripey Stripe"
